File: hardware/battleship_main_board/battleship_main_board.kicad_pcb (KiCad board)
At the start: 2 copper layers, 329 parts, among them J1 Conn_01x06, J2 Conn_01x06, SW1 SW_Push, SW10 SW_Push, SW100 SW_Push, SW11 SW_Push, SW12 SW_Push, SW13 SW_Push, SW14 SW_Push, SW15 SW_Push, SW16 SW_Push, SW17 SW_Push, SW18 SW_Push, SW19 SW_Push, SW2 SW_Push, SW20 SW_Push, SW21 SW_Push, SW22 SW_Push, SW23 SW_Push, SW24 SW_Push, SW25 SW_Push, SW26 SW_Push, SW27 SW_Push, SW28 SW_Push, SW29 SW_Push, SW3 SW_Push, SW30 SW_Push, SW31 SW_Push, SW32 SW_Push, SW33 SW_Push, SW34 SW_Push, SW35 SW_Push, SW36 SW_Push, SW37 SW_Push, SW38 SW_Push, SW39 SW_Push, SW4 SW_Push, SW40 SW_Push, SW41 SW_Push, SW42 SW_Push, SW43 SW_Push, SW44 SW_Push, SW45 SW_Push, SW46 SW_Push, SW47 SW_Push, SW48 SW_Push, SW49 SW_Push, SW5 SW_Push, SW50 SW_Push, SW51 SW_Push, SW52 SW_Push, SW53 SW_Push, SW54 SW_Push, SW55 SW_Push, SW56 SW_Push, SW57 SW_Push, SW58 SW_Push, SW59 SW_Push, SW6 SW_Push, SW60 SW_Push, SW61 SW_Push, SW62 SW_Push, SW63 SW_Push, SW64 SW_Push, SW65 SW_Push, SW66 SW_Push, SW67 SW_Push, SW68 SW_Push, SW69 SW_Push, SW7 SW_Push, SW70 SW_Push, SW71 SW_Push, SW72 SW_Push, SW73 SW_Push, SW74 SW_Push, SW75 SW_Push, SW76 SW_Push, SW77 SW_Push, SW78 SW_Push, SW79 SW_Push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

Commit message: updated pcb diagram
Parts:
- removed the U7 at (207.2, -405.3)
- moved LED22 649.1 mm to (-163.2, -145.3), turned to 180 degrees
- moved LED21 647.0 mm to (-178.2, -145.3), turned to 180 degrees
- moved LED42 630.4 mm to (-163.2, -115.3), turned to 180 degrees
- moved LED23 628.3 mm to (-148.2, -145.3), turned to 180 degrees
- moved LED41 628.1 mm to (-178.2, -115.3), turned to 180 degrees
- moved LED72 625.1 mm to (-163.2, -70.3), turned to 180 degrees
- moved LED24 622.1 mm to (-133.2, -145.3), turned to 180 degrees
- moved LED71 621.2 mm to (-178.2, -70.3), turned to 180 degrees
- moved LED43 609.5 mm to (-148.2, -115.3), turned to 180 degrees
- moved LED25 606.3 mm to (-118.2, -145.3), turned to 180 degrees
- moved LED73 603.9 mm to (-148.2, -70.3), turned to 180 degrees
- moved LED44 603.3 mm to (-133.2, -115.3), turned to 180 degrees
- moved LED74 598.2 mm to (-133.2, -70.3), turned to 180 degrees
- moved LED26 595.9 mm to (-103.2, -145.3), turned to 180 degrees
- moved LED28 588.6 mm to (-73.2, -145.3), turned to 180 degrees
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
Commit message: Finished routing
Parts:
- moved C1 131.7 mm to (30.5, -233.7)
- moved C5 107.0 mm to (106.7, -223.5)
- moved C2 91.5 mm to (15.3, -233.7)
- moved C6 90.5 mm to (127.0, -223.5)
- moved R2 82.7 mm to (114.3, -215.9)
- moved U1 78.9 mm to (-25.4, -228.6)
- moved U2 70.3 mm to (-8.88, -228.6)
- moved C7 66.0 mm to (132.1, -215.9)
- moved U3 64.1 mm to (7.62, -228.6)
- moved C3 61.6 mm to (7.62, -233.7), turned to 180 degrees
- moved U7 61.4 mm to (125.7, -203.2)
- moved U4 59.1 mm to (22.9, -228.6)
- moved D107 58.0 mm to (102.9, -188.0), turned to 180 degrees
- moved R1 55.5 mm to (-12.7, -233.7)
- moved D108 53.6 mm to (102.9, -195.6), turned to 180 degrees
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Routing:
- net GNDREF: track 0.00 -> 3298.8 mm, vias 0 -> 2
- net +5V: track 0.00 -> 3186.9 mm, vias 0 -> 4
- net /UserInputs/InputMatrix1/Row7: track 0.00 -> 364.6 mm, vias 0 -> 2
- net /UserInputs/InputMatrix1/Row9: track 0.00 -> 332.4 mm, vias 0 -> 4
- net /UserInputs/InputMatrix1/Row6: track 0.00 -> 322.0 mm, vias 0 -> 2
- net /UserInputs/InputMatrix1/Row8: track 0.00 -> 314.2 mm, vias 0 -> 3
- net /UserInputs/InputMatrix1/Row5: track 0.00 -> 305.6 mm, vias 0 -> 2
- net /UserInputs/InputMatrix1/Row4: track 0.00 -> 293.6 mm, vias 0 -> 2
- net /UserInputs/InputMatrix1/Row3: track 0.00 -> 279.9 mm, vias 0 -> 2
- net /UserInputs/InputMatrix1/Row2: track 0.00 -> 265.4 mm, vias 0 -> 2
- net /UserInputs/InputMatrix1/Row1: track 0.00 -> 252.8 mm, vias 0 -> 2
- net /ESP32/ButtonPressedIn: track 0.00 -> 226.8 mm
- net /ESP32/LED_out: track 0.00 -> 211.4 mm
- net /UserInputs/InputMatrix1/Row0: track 0.00 -> 204.0 mm, vias 0 -> 4
- net /ESP32/Clr: track 0.00 -> 201.8 mm, vias 0 -> 5
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